File: CESP.sch (KiCad schematic (older format))
At the start: 5 parts

Commit message: modified:   CESP-cache.lib new file:   CESP.cmp modified:   CESP.kicad_pcb modified:   CESP.kicad_pcb-bak new file:   CESP.net modified:   CESP.pro modified:   CESP.sch new file:   GLSP.lib new file:   GLSP.pretty/DPAK3.kicad_mod new file:   GLSP.pretty/FDMC8360L.kicad_mod new file:   GLSP.pretty/MCP6002.kicad_mod new file:   GLSP.pretty/TB62752AFUG.kicad_mod new file:   GLSP.pretty/ZXBM1021.kicad_mod new file:   Gerber/CESP-B_Cu.gbl new file:   Gerber/CESP-B_SilkS.gbo new file:   Gerber/CESP-F_Cu.gtl new file:   Gerber/CESP-F_SilkS.gto new file:   Gerber/CESP.drl new file:   fp-lib-table new file:   images/snapshot1.png new file:   images/snapshot2.png new file:   images/snapshot3.png
Parts:
- removed U?: LTC1594CS, TSSOP14, symbol LTC1594CS
- removed U?: TL074, TSSOP14, symbol TL074
- removed U? (x3): TL074, symbol TL074
- added C1, C3, C4: C, symbol C
- added R1, R3, R4: R, symbol R
- added U1: AO4576, symbol AO4576
- added U2: FDMC8360L, symbol FDMC8360L
- added U3: LM324, symbol LM324
- added U4: MCP6002, symbol MCP6002
- added U5: TB62752AFUG, symbol TB62752AFUG
- added U6: 7805, symbol 7805
Connections:
- net labels added: +5V, GND
- wire segments 0 -> 43
Other:
- note removed: "NOTE: THIS IS JUST A TEST BOARD\nREMOVE ALL COMPONENTS AND CREATE YOUR OWN\nINCLUDE SCHEMATIC HOOKUPS/NETLIST"
